Commit message: Add stage-one integer corridor-assignment learning pipeline.
Record planning instances, label MIQP assignments, and train optional BC/cost policies without baking weights into the planner. Center continuous AMPL variables, keep Gurobi NumericFocus/Presolve at defaults, and check residuals at 2e-6. Isolate stateCallback onto a mutually exclusive group to stop the actual-traj double-free. Capture protocol benchmark_aligned_v1 randomizes train/val starts and splits unknown-dynamic, static-forest, and privileged known-dynamic scenes. Fix D435 mesh lookup so depth is not empty.

This does not claim a learning benefit; aligned collection is still running.

File: urdf/_d435.urdf.xacro (robot description, xacro)
@@ -48,5 +48,5 @@
         <geometry>
           <!-- <box size="${d435_cam_width} ${d435_cam_height} ${d435_cam_depth}"/> -->
-          <mesh filename="package://sando/share/sando/meshes/real_sense/d435.dae" />
+          <mesh filename="$(find sando)/meshes/real_sense/d435.dae" />
         </geometry>
         <material name="${name}_aluminum"/>

File: urdf/_d435i.urdf.xacro (robot description, xacro)
@@ -69,5 +69,5 @@
       <origin xyz="${d435i_cam_mount_from_center_offset} ${-d435i_cam_depth_py} 0" rpy="${M_PI/2} 0 ${M_PI/2}"/>
         <geometry>
-          <mesh filename="package://sando/share/sando/meshes/real_sense/d435.dae"/>
+          <mesh filename="$(find sando)/meshes/real_sense/d435.dae"/>
         </geometry>
         <material name="${name}_aluminum"/>
